Commit message: update

File: urdf/rover_UT1.xacro (robot description, xacro)
@@ -5,7 +5,7 @@
   <link name="base_link">
     <visual>
-      <origin xyz="36.8 -5 -14.8" rpy="1.57 0 -1.57"/>
+      <origin xyz="3 13.75 -13.75" rpy="1.57 0 -1.57"/>
       <geometry>
-	      <mesh filename="package://rover_model/meshes/arm.dae"/>
+	      <mesh filename="package://rover_model/meshes/wheel_big.dae"/>
       </geometry>
     </visual>
@@ -23,5 +23,5 @@
     <parent link="base_link"/>
     <child link="test"/>
-    <origin xyz="30 0 0" rpy="0 0 0"/>
+    <origin xyz="160 100 0" rpy="0 0 0"/>
     <axis xyz="0 1 0"/>
     <dynamics damping="1"/>
